Commit message: KELO v2: two-layer map, people-aware navigation, driver views
- Two-layer map: Hokuyo LiDAR map plus a RealSense D435 camera layer
  (tables, shelves, overhangs), used in the global and local costmaps;
  camera layer can be rebuilt from the mapping bag on the finished map
- Navigation behaviour tree: stop, wait, then drive around an obstacle;
  people-aware waiting and passing (social node, IsPersonBlocking BT node)
- Robust localization: scan fit check, LOST detection, last pose restore
- Driver views: camera view with guide lines and planned path, surround
  view, object detection (YOLOX), coverage view, web view, video recorder
- robot_check: first-connection check of the robot interface
- GPU object detector service for the Jetson (TensorRT)
- Extended simulator and end-to-end tests

File: src/kelo_bringup/urdf/kelo.urdf.xacro (robot description, xacro)
@@ -5,4 +5,6 @@
   <xacro:arg name="camera_frame" default="camera_link"/>
   <xacro:arg name="camera_optical_frame" default="camera_depth_optical_frame"/>
+  <xacro:arg name="camera_color_optical_frame" default="camera_color_optical_frame"/>
+  <xacro:arg name="camera_color_y" default="0.0"/>
   <xacro:arg name="hedgehog_frame" default="hedgehog_link"/>
   <xacro:arg name="body_l" default="0.6"/>
@@ -47,4 +49,10 @@
     <origin xyz="0 0 0" rpy="-1.5707963267948966 0 -1.5707963267948966"/>
   </joint>
+  <link name="$(arg camera_color_optical_frame)"/>
+  <joint name="camera_to_color_optical" type="fixed">
+    <parent link="$(arg camera_frame)"/>
+    <child link="$(arg camera_color_optical_frame)"/>
+    <origin xyz="0 $(arg camera_color_y) 0" rpy="-1.5707963267948966 0 -1.5707963267948966"/>
+  </joint>
   <link name="$(arg hedgehog_frame)">
     <visual><geometry><cylinder radius="0.02" length="0.04"/></geometry><material name="orange"/></visual>
